Commit message: Fix diff drive plugin and wheel configuration
- Fix odometry_frame and robot_base_frame parameters
- Fix ROS remapping syntax
- Adjust wheel friction and damping parameters
- Fix spawn height to prevent robot sinking into ground

File: src/airobot_simulation/plugins/diff_drive.urdf.xacro (robot description, xacro)
@@ -51,4 +51,6 @@
 				<left_joint>${left_wheel}</left_joint>
 				<right_joint>${right_wheel}</right_joint>
+				<!-- 是否发布关节状态 -->
+				<publish_joint_state>true</publish_joint_state>
 				<!-- 运动学参数 -->
 				<!-- 左右轮间距 (米) -->
@@ -74,7 +76,7 @@
 				<!-- 坐标系 ID -->
 				<!-- 里程计坐标系 -->
-				<odom_frame_id>${odom_frame_id}</odom_frame_id>
+				<odometry_frame>${odom_frame_id}</odometry_frame>
 				<!-- 基座坐标系 -->
-				<base_frame_id>${base_frame_id}</base_frame_id>
+				<robot_base_frame>${base_frame_id}</robot_base_frame>
 				<!-- 世界坐标系 -->
 				<world_frame>${world_frame}</world_frame>

File: src/airobot_simulation/urdf/actuator/caster.urdf.xacro (robot description, xacro)
@@ -32,4 +32,11 @@
 			<origin xyz="${xyz}" rpy="0 0 0"/>
 		</joint>
+		<gazebo reference="${name}_link">
+			<material>Gazebo/Black</material>
+			<mu1>0.5</mu1>
+			<mu2>0.5</mu2>
+			<slip1>0.05</slip1>
+			<slip2>0.05</slip2>
+		</gazebo>
 	</xacro:macro>
 </robot>

File: src/airobot_simulation/urdf/actuator/wheel.urdf.xacro (robot description, xacro)
@@ -34,5 +34,11 @@
 			<origin xyz="${xyz}" rpy="0 0 0"/>
 			<axis xyz="0 1 0"/>
+			<dynamics damping="0.1" friction="0.1"/>
 		</joint>
+		<gazebo reference="${name}_link">
+			<material>Gazebo/DarkGrey</material>
+			<mu1>1.0</mu1>
+			<mu2>1.0</mu2>
+		</gazebo>
 	</xacro:macro>
 </robot>
