Commit message: Add Livox 3D LiDAR support with laser_type parameter
- Add laser_sensor_2d and laser_sensor_3d macros in laser.urdf.xacro
- 2D LiDAR: topic /scan, LaserScan message
- 3D LiDAR: topic /livox/lidar, PointCloud2 message
- Add laser_type parameter to airobot.urdf.xacro
- Remove non-existent rviz directory from airobot_cartographer CMakeLists

File: src/airobot_simulation/plugins/laser.urdf.xacro (robot description, xacro)
@@ -3,7 +3,11 @@
 	<!--
 	激光雷达传感器插件 (Laser Sensor Plugin) 用于 Gazebo 仿真
+	支持两种类型:
+	- laser_type:="2d" - 传统2D激光雷达 (默认)
+	- laser_type:="3d" - Livox 3D激光雷达
 	参数说明:
 	- name: 传感器名称
 	- parent: 父链接名称
+	- laser_type: 激光雷达类型 (2d 或 3d, 默认: 2d)
 	- topic_name: 激光扫描数据发布的话题名称 (默认: scan)
 	- frame_id: 传感器坐标系 ID (默认: laser_link)
@@ -15,24 +19,25 @@
 	- ray_angle_min: 最小扫描角度 (弧度, 默认: -3.14159)
 	- ray_angle_max: 最大扫描角度 (弧度, 默认: 3.14159)
-	- ray_angle_increment: 角度增量 (弧度, 默认: 0.0175)
-	-xyz: 传感器相对于父链接的位置 (默认: 0 0 0)
+	- xyz: 传感器相对于父链接的位置 (默认: 0 0 0)
 	- rpy: 传感器的姿态 (默认: 0 0 0)
-	- publish_tf: 是否发布 TF (默认: true)
 	- visualize: 是否显示激光扫描可视化 (默认: true)
 	- always_on: 传感器是否始终启用 (默认: true)
-	-->
-	<!--
-	完整版激光雷达插件宏
-	包含所有可配置参数
-	-->
-	<xacro:macro name="laser_sensor" params="name parent
+	3D (Livox) 专用参数:
+	- vertical_samples: 垂直射线数量 (默认: 16)
+	- vertical_angle_min: 最小垂直角度 (弧度, 默认: -0.523 = -30°)
+	- vertical_angle_max: 最大垂直角度 (弧度, 默认: 0.523 = 30°)
+	-->
+	<!--
+	2D 激光雷达插件宏
+	-->
+	<xacro:macro name="laser_sensor_2d" params="name parent
 		topic_name:='scan'
 		update_rate:=10
 		ray_count:=360
 		ray_range_min:=0.10 ray_range_max:=10.0 ray_range_resolution:=0.01
-		ray_angle_min:=-3.14159 ray_angle_max:=3.14159 ray_angle_increment:=0.0175
+		ray_angle_min:=-3.14159 ray_angle_max:=3.14159
 		xyz:='0 0 0' rpy:='0 0 0'
-		publish_tf:=true visualize:=true always_on:=true">
-		<!-- Gazebo 激光雷达传感器插件 -->
+		visualize:=true always_on:=true">
+		<!-- Gazebo 2D 激光雷达传感器插件 -->
 		<gazebo reference="${name}_link">
 			<pose>${xyz} ${rpy}</pose>
@@ -44,5 +49,5 @@
 				<always_on>${always_on}</always_on>
 				<visualize>${visualize}</visualize>
-				<!-- 激光射线配置 -->
+				<!-- 2D 激光射线配置 (只有水平扫描) -->
 				<ray>
 					<scan>
@@ -73,5 +78,5 @@
 					<!-- 话题设置 -->
 					<topic_name>${topic_name}</topic_name>
-					<!-- 输出类型 -->
+					<!-- 输出类型: 2D LaserScan -->
 					<output_type>sensor_msgs/LaserScan</output_type>
 					<!-- 坐标系 -->
@@ -82,13 +87,135 @@
 	</xacro:macro>
 	<!--
-	简化版激光雷达插件宏
-	只包含必要参数，其他使用默认值
-	-->
-	<xacro:macro name="laser_sensor_simple" params="name parent topic_name:='scan' update_rate:=10
+	Livox 3D 激光雷达插件宏
+	支持 Livox Horizon, Mid-40, Mid-70 等型号
+	-->
+	<xacro:macro name="laser_sensor_3d" params="name parent
+		topic_name:='livox/lidar'
+		update_rate:=10
+		ray_range_min:=0.10 ray_range_max:=90.0 ray_range_resolution:=0.01
+		horizontal_samples:=1920
+		horizontal_angle_min:=-0.674 horizontal_angle_max:=0.674
+		vertical_samples:=16
+		vertical_angle_min:=-0.523 vertical_angle_max:=0.523
+		xyz:='0 0 0' rpy:='0 0 0'
+		visualize:=true always_on:=true">
+		<!-- Gazebo 3D 激光雷达传感器插件 -->
+		<gazebo reference="${name}_link">
+			<pose>${xyz} ${rpy}</pose>
+			<sensor type="gpu_ray" name="${name}">
+				<pose>0 0 0 0 0 0</pose>
+				<!-- 更新频率 (Hz) -->
+				<update_rate>${update_rate}</update_rate>
+				<!-- 视觉和碰撞设置 -->
+				<always_on>${always_on}</always_on>
+				<visualize>${visualize}</visualize>
+				<!-- 3D 激光射线配置 (水平和垂直扫描) -->
+				<ray>
+					<scan>
+						<horizontal>
+							<samples>${horizontal_samples}</samples>
+							<resolution>1</resolution>
+							<min_angle>${horizontal_angle_min}</min_angle>
+							<max_angle>${horizontal_angle_max}</max_angle>
+						</horizontal>
+						<vertical>
+							<samples>${vertical_samples}</samples>
+							<resolution>1</resolution>
+							<min_angle>${vertical_angle_min}</min_angle>
+							<max_angle>${vertical_angle_max}</max_angle>
+						</vertical>
+					</scan>
+					<range>
+						<min>${ray_range_min}</min>
+						<max>${ray_range_max}</max>
+						<resolution>${ray_range_resolution}</resolution>
+					</range>
+					<noise>
+						<type>gaussian</type>
+						<mean>0.0</mean>
+						<stddev>0.01</stddev>
+					</noise>
+				</ray>
+				<!-- 插件配置 -->
+				<plugin name="${name}_plugin" filename="libgazebo_ros_ray_sensor.so">
+					<ros>
+						<namespace>/</namespace>
+						<remapping>~/out:=${topic_name}</remapping>
+					</ros>
+					<!-- 话题设置 -->
+					<topic_name>${topic_name}</topic_name>
+					<!-- 输出类型: 3D PointCloud2 -->
+					<output_type>sensor_msgs/PointCloud2</output_type>
+					<!-- 坐标系 -->
+					<frame_name>${name}_link</frame_name>
+				</plugin>
+			</sensor>
+		</gazebo>
+	</xacro:macro>
+	<!--
+	统一激光雷达宏 - 根据 laser_type 参数自动选择 2D 或 3D
+	laser_type:="2d" 或 laser_type:="3d"
+	-->
+	<xacro:macro name="laser_sensor" params="name parent
+		laser_type:='2d'
+		topic_name:='scan'
+		update_rate:=10
+		ray_count:=360
+		ray_range_min:=0.10 ray_range_max:=10.0 ray_range_resolution:=0.01
+		ray_angle_min:=-3.14159 ray_angle_max:=3.14159
+		horizontal_samples:=1920 horizontal_angle_min:=-0.674 horizontal_angle_max:=0.674
+		vertical_samples:=16 vertical_angle_min:=-0.523 vertical_angle_max:=0.523
+		xyz:='0 0 0' rpy:='0 0 0'
+		visualize:=true always_on:=true">
+		<!-- 根据 laser_type 选择对应的传感器宏 -->
+		<xacro:if value="${laser_type == '2d'}">
+			<xacro:laser_sensor_2d
+				name="${name}"
+				parent="${parent}"
+				topic_name="${topic_name}"
+				update_rate="${update_rate}"
+				ray_count="${ray_count}"
+				ray_range_min="${ray_range_min}"
+				ray_range_max="${ray_range_max}"
+				ray_range_resolution="${ray_range_resolution}"
+				ray_angle_min="${ray_angle_min}"
+				ray_angle_max="${ray_angle_max}"
+				xyz="${xyz}"
+				rpy="${rpy}"
+				visualize="${visualize}"
+				always_on="${always_on}"/>
+		</xacro:if>
+		<xacro:if value="${laser_type == '3d'}">
+			<xacro:laser_sensor_3d
+				name="${name}"
+				parent="${parent}"
+				topic_name="${topic_name}"
+				update_rate="${update_rate}"
+				ray_range_min="${ray_range_min}"
+				ray_range_max="${ray_range_max}"
+				ray_range_resolution="${ray_range_resolution}"
+				horizontal_samples="${horizontal_samples}"
+				horizontal_angle_min="${horizontal_angle_min}"
+				horizontal_angle_max="${horizontal_angle_max}"
+				vertical_samples="${vertical_samples}"
+				vertical_angle_min="${vertical_angle_min}"
+				vertical_angle_max="${vertical_angle_max}"
+				xyz="${xyz}"
+				rpy="${rpy}"
+				visualize="${visualize}"
+				always_on="${always_on}"/>
+		</xacro:if>
+	</xacro:macro>
+	<!--
+	简化版激光雷达插件宏 - 只包含必要参数
+	默认使用 2D 激光雷达
+	-->
+	<xacro:macro name="laser_sensor_simple" params="name parent laser_type:='2d' topic_name:='scan' update_rate:=10
 		ray_range_min:=0.10 ray_range_max:=10.0 xyz:='0 0 0' rpy:='0 0 0' always_on:=true">
-		<!-- 调用完整版宏，使用默认参数 -->
+		<!-- 调用统一宏 -->
 		<xacro:laser_sensor
 			name="${name}"
 			parent="${parent}"
+			laser_type="${laser_type}"
 			topic_name="${topic_name}"
 			update_rate="${update_rate}"

File: src/airobot_simulation/urdf/airobot/airobot.urdf.xacro (robot description, xacro)
@@ -29,9 +29,10 @@
 		camera_type: 相机类型 (rgb: 普通相机, depth: 深度相机) (默认: rgb)
 		imu_xyz: IMU相对于基座的安装位置(x,y,z,单位:米)
+		laser_type: 激光雷达类型 (2d: 2D激光雷达, 3d: Livox 3D激光雷达) (默认: 2d)
 		laser_xyz: 激光雷达相对于基座的安装位置(x,y,z,单位:米)
 		laser_angle_min: 激光雷达最小扫描角度(弧度)
 		laser_angle_max: 激光雷达最大扫描角度(弧度)
 	-->
-	<xacro:macro name="airobot" params="base_length base_radius left_wheel_xyz right_wheel_xyz rear_caster_xyz front_caster_xyz camera_xyz camera_type imu_xyz laser_xyz laser_angle_min laser_angle_max">
+	<xacro:macro name="airobot" params="base_length base_radius left_wheel_xyz right_wheel_xyz rear_caster_xyz front_caster_xyz camera_xyz camera_type imu_xyz laser_type laser_xyz laser_angle_min laser_angle_max">
 		<!-- 基座足印链接(虚拟链接,用于确定机器人底部位置) -->
 		<link name="base_footprint"/>
@@ -66,10 +67,13 @@
 		<!-- 激光雷达传感器 -->
 		<xacro:laser name="laser" parent="base_link" xyz="${laser_xyz}"/>
+		<!-- 根据激光雷达类型设置不同的话题名称 -->
+		<xacro:property name="laser_topic" value="${'livox/lidar' if laser_type == '3d' else 'scan'}"/>
 		<!-- 激光雷达传感器插件 -->
-		<!-- 参数: name(传感器名称), parent(父链接), topic_name(发布话题名), update_rate(更新频率Hz), xyz(安装位置) -->
+		<!-- 参数: name(传感器名称), parent(父链接), laser_type(激光雷达类型), topic_name(发布话题名), update_rate(更新频率Hz), xyz(安装位置) -->
 		<xacro:laser_sensor
 			name="laser"
 			parent="base_link"
-			topic_name="scan"
+			laser_type="${laser_type}"
+			topic_name="${laser_topic}"
 			update_rate="10"
 			visualize="false"
@@ -109,4 +113,5 @@
 	<xacro:arg name="camera_type" default="depth"/>           <!-- 相机类型: rgb=普通相机, depth=深度相机 -->
 	<xacro:arg name="imu_xyz" default="0.0 0.0 0.03"/>       <!-- IMU安装位置(x y z,单位:米) -->
+	<xacro:arg name="laser_type" default="3d"/>           <!-- 激光雷达类型: 2d=2D激光雷达, 3d=Livox 3D激光雷达 -->
 	<xacro:arg name="laser_xyz" default="0.0 0.0 0.125"/>   <!-- 激光雷达安装位置(x y z,单位:米) -->
 	<!-- 激光雷达扫描角度参数 -->
@@ -127,4 +132,5 @@
 			camera_type="$(arg camera_type)"
 			imu_xyz="$(arg imu_xyz)"
+			laser_type="$(arg laser_type)"
 			laser_xyz="$(arg laser_xyz)"
 			laser_angle_min="$(arg laser_angle_min)"
