Commit message: 为URDF和插件文件添加中文注释
- actuator/caster.urdf.xacro: 添加从动轮参数中文注释
- actuator/wheel.urdf.xacro: 添加车轮参数中文注释
- airobot/base.urdf.xacro: 添加基座参数中文注释
- sensor/camera.urdf.xacro: 添加摄像头参数中文注释
- sensor/imu.urdf.xacro: 添加IMU参数中文注释
- sensor/laser.urdf.xacro: 添加激光雷达参数中文注释

File: src/airobot_simulation/urdf/actuator/caster.urdf.xacro (robot description, xacro)
@@ -1,8 +1,11 @@
 <?xml version="1.0"?>
 <robot xmlns:xacro="http://www.ros.org/wiki/xacro" name="caster_macro">
+	<!-- 从动轮(万向轮)执行器宏定义 -->
+	<!-- 参数: name(从动轮名称), parent(父链接), xyz(安装位置) -->
 	<xacro:macro name="caster" params="name parent xyz">
-		<xacro:property name="caster_radius" value="0.04"/>
-		<xacro:property name="caster_mass" value="0.3"/>
-		<xacro:property name="caster_inertia" value="${0.4 * caster_mass * caster_radius * caster_radius}"/>
+		<!-- 从动轮参数 -->
+		<xacro:property name="caster_radius" value="0.04"/>      <!-- 从动轮半径(米) -->
+		<xacro:property name="caster_mass" value="0.3"/>         <!-- 从动轮质量(千克) -->
+		<xacro:property name="caster_inertia" value="${0.4 * caster_mass * caster_radius * caster_radius}"/>  <!-- 惯性矩 -->
 		<link name="${name}_link">
 			<visual>

File: src/airobot_simulation/urdf/actuator/wheel.urdf.xacro (robot description, xacro)
@@ -1,8 +1,12 @@
 <?xml version="1.0"?>
 <robot xmlns:xacro="http://www.ros.org/wiki/xacro" name="wheel_macro">
+	<!-- 车轮执行器宏定义 -->
+	<!-- 参数: name(车轮名称), parent(父链接), xyz(安装位置) -->
 	<xacro:macro name="wheel" params="name parent xyz">
-		<xacro:property name="wheel_radius" value="0.08"/>
-		<xacro:property name="wheel_width" value="0.04"/>
-		<xacro:property name="wheel_mass" value="0.8"/>
+		<!-- 车轮参数 -->
+		<xacro:property name="wheel_radius" value="0.08"/>      <!-- 车轮半径(米) -->
+		<xacro:property name="wheel_width" value="0.04"/>      <!-- 车轮宽度(米) -->
+		<xacro:property name="wheel_mass" value="0.8"/>         <!-- 车轮质量(千克) -->
+		<!-- 车轮惯性矩计算 -->
 		<xacro:property name="wheel_ixx" value="${wheel_mass * (3.0 * wheel_radius * wheel_radius + wheel_width * wheel_width) / 12.0}"/>
 		<xacro:property name="wheel_izz" value="${0.5 * wheel_mass * wheel_radius * wheel_radius}"/>

File: src/airobot_simulation/urdf/airobot/base.urdf.xacro (robot description, xacro)
@@ -1,6 +1,10 @@
 <?xml version="1.0"?>
 <robot xmlns:xacro="http://www.ros.org/wiki/xacro" name="base_macro">
+	<!-- 机器人基座宏定义 -->
+	<!-- 参数: name(基座名称), length(基座长度/高度), radius(基座半径) -->
 	<xacro:macro name="base" params="name length radius">
-		<xacro:property name="base_mass" value="8.0"/>
+		<!-- 基座物理参数 -->
+		<xacro:property name="base_mass" value="8.0"/>    <!-- 基座质量(千克) -->
+		<!-- 基座惯性矩计算 -->
 		<xacro:property name="base_ixx" value="${base_mass * (3.0 * radius * radius + length * length) / 12.0}"/>
 		<xacro:property name="base_izz" value="${0.5 * base_mass * radius * radius}"/>

File: src/airobot_simulation/urdf/sensor/camera.urdf.xacro (robot description, xacro)
@@ -1,9 +1,12 @@
 <?xml version="1.0"?>
 <robot xmlns:xacro="http://www.ros.org/wiki/xacro" name="camera_macro">
+	<!-- 摄像头传感器宏定义 -->
+	<!-- 参数: name(传感器名称), parent(父链接), xyz(安装位置) -->
 	<xacro:macro name="camera" params="name parent xyz">
-		<xacro:property name="camera_mass" value="0.15"/>
-		<xacro:property name="camera_x" value="0.06"/>
-		<xacro:property name="camera_y" value="0.03"/>
-		<xacro:property name="camera_z" value="0.03"/>
+		<!-- 摄像头参数 -->
+		<xacro:property name="camera_mass" value="0.15"/>  <!-- 摄像头质量(千克) -->
+		<xacro:property name="camera_x" value="0.06"/>    <!-- 摄像头X尺寸(米) -->
+		<xacro:property name="camera_y" value="0.03"/>    <!-- 摄像头Y尺寸(米) -->
+		<xacro:property name="camera_z" value="0.03"/>     <!-- 摄像头Z尺寸(米) -->
 		<link name="${name}_link">
 			<visual>

File: src/airobot_simulation/urdf/sensor/imu.urdf.xacro (robot description, xacro)
@@ -1,7 +1,10 @@
 <?xml version="1.0"?>
 <robot xmlns:xacro="http://www.ros.org/wiki/xacro" name="imu_macro">
+	<!-- IMU(惯性测量单元)传感器宏定义 -->
+	<!-- 参数: name(传感器名称), parent(父链接), xyz(安装位置) -->
 	<xacro:macro name="imu" params="name parent xyz">
-		<xacro:property name="imu_mass" value="0.05"/>
-		<xacro:property name="imu_size" value="0.025"/>
+		<!-- IMU参数 -->
+		<xacro:property name="imu_mass" value="0.05"/>      <!-- IMU质量(千克) -->
+		<xacro:property name="imu_size" value="0.025"/>    <!-- IMU尺寸(米,立方体边长) -->
 		<link name="${name}_link">
 			<visual>

File: src/airobot_simulation/urdf/sensor/laser.urdf.xacro (robot description, xacro)
@@ -1,11 +1,15 @@
 <?xml version="1.0"?>
 <robot xmlns:xacro="http://www.ros.org/wiki/xacro" name="laser_macro">
+	<!-- 激光雷达传感器宏定义 -->
+	<!-- 参数: name(传感器名称), parent(父链接), xyz(安装位置) -->
 	<xacro:macro name="laser" params="name parent xyz">
-		<xacro:property name="pole_radius" value="0.01"/>
-		<xacro:property name="pole_height" value="0.10"/>
-		<xacro:property name="pole_mass" value="0.08"/>
-		<xacro:property name="laser_radius" value="0.04"/>
-		<xacro:property name="laser_height" value="0.05"/>
-		<xacro:property name="laser_mass" value="0.2"/>
+		<!-- 支架参数 -->
+		<xacro:property name="pole_radius" value="0.01"/>   <!-- 支架半径(米) -->
+		<xacro:property name="pole_height" value="0.10"/>  <!-- 支架高度(米) -->
+		<xacro:property name="pole_mass" value="0.08"/>    <!-- 支架质量(千克) -->
+		<!-- 激光雷达参数 -->
+		<xacro:property name="laser_radius" value="0.04"/>  <!-- 激光雷达半径(米) -->
+		<xacro:property name="laser_height" value="0.05"/>  <!-- 激光雷达高度(米) -->
+		<xacro:property name="laser_mass" value="0.2"/>     <!-- 激光雷达质量(千克) -->
 		<link name="${name}_mount_link">
 			<visual>
